Commit message: test astar

File: urdf/turtlebot3_waffle_pi.gazebo.xacro (robot description, xacro)
@@ -46,46 +46,18 @@
     <material>Gazebo/FlatBlack</material>
   </gazebo>
-  <!-- <gazebo reference="imu_link">
-    <sensor type="imu" name="imu">
-      <always_on>true</always_on>
-      <visualize>$(arg imu_visual)</visualize>
-    </sensor>
-    <material>Gazebo/Grey</material>
-  </gazebo> -->
   <gazebo>
     <plugin name="turtlebot3_waffle_pi_controller" filename="libgazebo_ros_diff_drive.so">
-      <!-- <commandTopic>cmd_vel</commandTopic>
-      <odometryTopic>odom</odometryTopic>
-      <odometryFrame>odom</odometryFrame>
-      <odometrySource>world</odometrySource>
-      <publishOdomTF>true</publishOdomTF>
-      <robotBaseFrame>base_footprint</robotBaseFrame>
-      <publishWheelTF>false</publishWheelTF>
-      <publishTf>true</publishTf>
-      <publishWheelJointState>true</publishWheelJointState>
-      <legacyMode>false</legacyMode>
-      <updateRate>30</updateRate>
-      <leftJoint>wheel_left_joint</leftJoint>
-      <rightJoint>wheel_right_joint</rightJoint>
-      <wheelSeparation>0.287</wheelSeparation>
-      <wheelDiameter>0.066</wheelDiameter>
-      <wheelAcceleration>1</wheelAcceleration>
-      <wheelTorque>10</wheelTorque>
-      <rosDebugLevel>na</rosDebugLevel> -->
-      <!-- <ros>
-        <namespace>/tb3_0</namespace>
-      </ros> -->
+      <ros>
+        <namespace>$(arg namespace)</namespace>
+        <argument>--ros-args -p use_sim_time:=true</argument>
+      </ros>
       <update_rate>30</update_rate>
-      <!-- wheels -->
       <left_joint>wheel_left_joint</left_joint>
       <right_joint>wheel_right_joint</right_joint>
-      <!-- kinematics -->
       <wheel_separation>0.287</wheel_separation>
       <wheel_diameter>0.066</wheel_diameter>
-      <!-- limits -->
       <max_wheel_torque>20</max_wheel_torque>
       <max_wheel_acceleration>1.0</max_wheel_acceleration>
       <command_topic>cmd_vel</command_topic>
-      <!-- output -->
       <publish_odom>true</publish_odom>
       <publish_odom_tf>true</publish_odom_tf>
@@ -94,15 +66,9 @@
       <odometry_frame>/$(arg namespace)/odom</odometry_frame>
       <robot_base_frame>/$(arg namespace)/base_footprint</robot_base_frame>
-      <!-- <left_joint>wheel_left_joint</left_joint>
-      <right_joint>wheel_right_joint</right_joint>
-      <wheel_separation>0.287</wheel_separation>
-      <wheel_radius>0.033</wheel_radius>
-      <odom_publish_frequency>1</odom_publish_frequency>
-      <topic>cmd_vel</topic> -->
     </plugin>
     <plugin name="turtlebot3_joint_state" filename="libgazebo_ros_joint_state_publisher.so">
       <ros>
-        <!-- <namespace>${namespace}</namespace> -->
         <remapping>~/out:=joint_states</remapping>
+        <argument>--ros-args -p use_sim_time:=true</argument>
       </ros>
       <update_rate>30</update_rate>
@@ -113,30 +79,4 @@
   <gazebo reference="imu_link">
     <material>Gazebo/Grey</material>
-    <!-- <plugin name="imu_plugin" filename="libgazebo_ros_imu.so">
-      <alwaysOn>true</alwaysOn>
-      <bodyName>imu_link</bodyName>
-      <frameName>imu_link</frameName>
-      <topicName>imu</topicName>
-      <serviceName>imu_service</serviceName>
-      <gaussianNoise>0.0</gaussianNoise>
-      <updateRate>0</updateRate>
-      <imu>
-        <noise>
-          <type>gaussian</type>
-          <rate>
-            <mean>0.0</mean>
-            <stddev>2e-4</stddev>
-            <bias_mean>0.0000075</bias_mean>
-            <bias_stddev>0.0000008</bias_stddev>
-          </rate>
-          <accel>
-            <mean>0.0</mean>
-            <stddev>1.7e-2</stddev>
-            <bias_mean>0.1</bias_mean>
-            <bias_stddev>0.001</bias_stddev>
-          </accel>
-        </noise>
-      </imu>
-    </plugin> -->
     <sensor name="tb3_imu" type="imu">
         <always_on>true</always_on>
@@ -187,6 +127,6 @@
         <plugin name="turtlebot3_imu" filename="libgazebo_ros_imu_sensor.so">
           <ros>
-            <!-- <namespace>${namespace}</namespace> -->
             <remapping>~/out:=imu</remapping>
+            <argument>--ros-args -p use_sim_time:=true</argument>
           </ros>
         </plugin>
@@ -195,33 +135,4 @@
   <gazebo reference="base_scan">
     <material>Gazebo/FlatBlack</material>
-    <!-- <sensor type="ray" name="lds_lfcd_sensor">
-      <pose>0 0 0 0 0 0</pose>
-      <visualize>$(arg laser_visual)</visualize>
-      <update_rate>5</update_rate>
-      <ray>
-        <scan>
-          <horizontal>
-            <samples>360</samples>
-            <resolution>1</resolution>
-            <min_angle>0.0</min_angle>
-            <max_angle>6.28319</max_angle>
-          </horizontal>
-        </scan>
-        <range>
-          <min>0.120</min>
-          <max>3.5</max>
-          <resolution>0.015</resolution>
-        </range>
-        <noise>
-          <type>gaussian</type>
-          <mean>0.0</mean>
-          <stddev>0.01</stddev>
-        </noise>
-      </ray>
-      <plugin name="gazebo_ros_lds_lfcd_controller" filename="libgazebo_ros_laser.so">
-        <topicName>scan</topicName>
-        <frameName>base_scan</frameName>
-      </plugin>
-    </sensor> -->
     <sensor name="hls_lfcd_lds" type="ray">
       <always_on>true</always_on>
@@ -251,6 +162,6 @@
       <plugin name="turtlebot3_laserscan" filename="libgazebo_ros_ray_sensor.so">
         <ros>
-          <!-- <namespace>${namespace}</namespace> -->
           <remapping>~/out:=scan</remapping>
+          <argument>--ros-args -p use_sim_time:=true</argument>
         </ros>
         <output_type>sensor_msgs/LaserScan</output_type>
@@ -259,70 +170,31 @@
     </sensor>
   </gazebo>
-<!--link : https://www.raspberrypi.org/documentation/hardware/camera/-->
-  <gazebo reference="camera_rgb_frame">
-    <!-- <sensor type="camera" name="pi_camera">
+<gazebo reference="camera_rgb_frame">
+    <sensor name="camera" type="camera">
       <always_on>true</always_on>
       <visualize>$(arg camera_visual)</visualize>
-      <camera>
-          <horizontal_fov>1.085595</horizontal_fov>
-          <image>
-              <width>640</width>
-              <height>480</height>
-              <format>R8G8B8</format>
-          </image>
-          <clip>
-              <near>0.03</near>
-              <far>100</far>
-          </clip>
+      <update_rate>30</update_rate>
+      <camera name="picam">
+        <horizontal_fov>1.085595</horizontal_fov>
+        <image>
+            <width>640</width>
+            <height>480</height>
+            <format>R8G8B8</format>
+        </image>
+        <clip>
+            <near>0.03</near>
+            <far>100</far>
+        </clip>
+        <noise>
+          <type>gaussian</type>
+          <mean>0.0</mean>
+          <stddev>0.007</stddev>
+        </noise>
       </camera>
-      <plugin name="camera_controller" filename="libgazebo_ros_camera.so">
-        <alwaysOn>true</alwaysOn>
-        <updateRate>30.0</updateRate>
-        <cameraName>camera</cameraName>
-        <frameName>camera_rgb_optical_frame</frameName>
-        <imageTopicName>rgb/image_raw</imageTopicName>
-        <cameraInfoTopicName>rgb/camera_info</cameraInfoTopicName>
-        <hackBaseline>0.07</hackBaseline>
-        <distortionK1>0.0</distortionK1>
-        <distortionK2>0.0</distortionK2>
-        <distortionK3>0.0</distortionK3>
-        <distortionT1>0.0</distortionT1>
-        <distortionT2>0.0</distortionT2>
-      </plugin>
-    </sensor> -->
-    <sensor name="camera" type="camera">
-        <always_on>true</always_on>
-        <visualize>$(arg camera_visual)</visualize>
-        <update_rate>30</update_rate>
-        <camera name="picam">
-          <horizontal_fov>1.085595</horizontal_fov>
-          <image>
-              <width>640</width>
-              <height>480</height>
-              <format>R8G8B8</format>
-          </image>
-          <clip>
-              <near>0.03</near>
-              <far>100</far>
-          </clip>
-          <noise>
-            <type>gaussian</type>
-            <!-- Noise is sampled independently per pixel on each frame.
-                  That pixel's noise value is added to each of its color
-                  channels, which at that point lie in the range [0,1]. -->
-            <mean>0.0</mean>
-            <stddev>0.007</stddev>
-          </noise>
-        </camera>
-          <plugin name="camera_driver" filename="libgazebo_ros_camera.so">
-            <ros>
-              <!-- <namespace>test_cam</namespace> -->
-              <!-- <remapping>image_raw:=image_demo</remapping> -->
-              <!-- <remapping>camera_info:=camera_info_demo</remapping> -->
-            </ros>
-            <!-- camera_name>omit so it defaults to sensor name</camera_name-->
-            <!-- frame_name>omit so it defaults to link name</frameName-->
-            <!-- <hack_baseline>0.07</hack_baseline> -->
-          </plugin>
+        <plugin name="camera_driver" filename="libgazebo_ros_camera.so">
+          <ros>
+            <argument>--ros-args -p use_sim_time:=true</argument>
+          </ros>
+        </plugin>
       </sensor>
   </gazebo>
